File: board/PCB_Bot.kicad_pcb (KiCad board)
At the start: 2 copper layers, 18 parts, among them J1 Screw_Terminal_01x04, J2 Conn_02x15_Top_Bottom, J3 Conn_02x15_Top_Bottom, J4 Screw_Terminal_01x02, J5 Screw_Terminal_01x03, U1 TB6612FNG, U2 LSM9DS1

Commit message: update pcbnew orienatation
Parts:
- moved J2 17.8 mm to (91.4, 72.4)
- moved J3 17.8 mm to (109.2, 72.4)
- moved C1 0.07 mm to (99.6, 85.8)
Connections:
- J3 pad 5: RST -> RST1
- J3 pad 6: RST -> RST1
Routing:
- net RST: track 5.08 -> 0.00 mm
- net GND: track 5.08 -> 0.00 mm
- net VIN: track 2.54 -> 0.00 mm
- net TX1: track 2.54 -> 0.00 mm
- net RX0: track 2.54 -> 0.00 mm
- net REF: track 2.54 -> 0.00 mm
- net D9: track 2.54 -> 0.00 mm
- net D8: track 2.54 -> 0.00 mm
- net D7: track 2.54 -> 0.00 mm
- net D6: track 2.54 -> 0.00 mm
- net D5: track 2.54 -> 0.00 mm
- net D4: track 2.54 -> 0.00 mm
- net D3: track 2.54 -> 0.00 mm
- net D2: track 2.54 -> 0.00 mm
- net D13: track 2.54 -> 0.00 mm
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Other:
- board outline added: 34.5 x 40.1 mm
Changed lines of the file:
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@@
   (general
     (thickness 1.6)
-    (drawings 0)
-    (tracks 33)
+    (drawings 4)
+    (tracks 0)
     (zones 0)
     (modules 18)
-    (nets 40)
+    (nets 41)
   )
   (page A4)
@@
     (solder_mask_min_width 0.25)
     (aux_axis_origin 0 0)
-    (visible_elements 7FFFFFFF)
+    (grid_origin 86.7918 110.109)
+    (visible_elements 7FFDFFFF)
     (pcbplotparams
       (layerselection 0x010fc_ffffffff)
@@
   (net 38 REF)
   (net 39 D13)
+  (net 40 RST1)
   (net_class Default "This is the default net class."
     (clearance 0.2)
@@
     (add_net REF)
     (add_net RST)
+    (add_net RST1)
     (add_net RX0)
     (add_net TX1)
@@
     (tags "LGA 24L 3x3.5mm Pitch 0.43mm")
     (attr smd)
-    (fp_text reference U2 (at 0 -2.7) (layer F.SilkS)
-      (effects (font (size 1 1) (thickness 0.15)))
-    )
-    (fp_text value LSM9DS1 (at 0 2.8) (layer F.Fab)
+    (fp_text reference U2 (at 1.3462 2.7432) (layer F.SilkS)
+      (effects (font (size 1 1) (thickness 0.15)))
+    )
+    (fp_text value LSM9DS1 (at 0 2.8) (layer F.Fab) hide
       (effects (font (size 1 1) (thickness 0.15)))
     )
@@
   )
   (module Connector_PinSocket_2.54mm:PinSocket_2x15_P2.54mm_Vertical (layer F.Cu)
-    (at 109.22 72.39)
+    (at 91.44 72.39)
     (descr "Through hole straight socket strip, 2x15, 2.54mm pitch, double cols (from Kicad 4.0.7), script generated")
     (tags "Through hole socket strip THT 2x15 2.54mm double row")
-    (fp_text reference J2 (at -1.27 -2.77) (layer F.SilkS)
+    (fp_text reference J2 (at -5.6642 -0.4826) (layer F.SilkS)
       (effects (font (size 1 1) (thickness 0.15)))
     )
@@
   )
   (module Capacitor_SMD:C_0603_1608Metric (layer F.Cu)
-    (at 99.695 85.725 270)
+    (at 99.6442 85.7757 270)
     (descr "Capacitor SMD 0603 (1608 Metric), square (rectangular) end terminal, IPC_7351 nominal, (Body size source: http://www.tortai-tech.com/upload/download/2011102023233369053.pdf), generated with kicad-footprint-generator")
     (tags capacitor)
     (attr smd)
-    (fp_text reference C1 (at 0 -1.43 90) (layer F.SilkS)
+    (fp_text reference C1 (at 2.4384 -0.0254 90) (layer F.SilkS)
       (effects (font (size 1 1) (thickness 0.15)))
     )
@@
     (tags capacitor)
     (attr smd)
-    (fp_text reference C2 (at 0 -1.65 90) (layer F.SilkS)
+    (fp_text reference C2 (at 2.6924 -0.1524 90) (layer F.SilkS)
       (effects (font (size 1 1) (thickness 0.15)))
     )
@@
     (tags capacitor)
     (attr smd)
-    (fp_text reference C3 (at 0 -1.43 90) (layer F.SilkS)
+    (fp_text reference C3 (at 2.54 -0.0762 90) (layer F.SilkS)
       (effects (font (size 1 1) (thickness 0.15)))
     )
@@
     (tags capacitor)
     (attr smd)
-    (fp_text reference C4 (at 0 -1.65 90) (layer F.SilkS)
+    (fp_text reference C4 (at 2.6924 0.1778 90) (layer F.SilkS)
       (effects (font (size 1 1) (thickness 0.15)))
     )
@@
     (tags capacitor)
     (attr smd)
-    (fp_text reference C5 (at 0 -1.65) (layer F.SilkS)
+    (fp_text reference C5 (at 2.8702 -0.127) (layer F.SilkS)
       (effects (font (size 1 1) (thickness 0.15)))
     )
@@
     (tags capacitor)
     (attr smd)
-    (fp_text reference C6 (at 0 -1.43 90) (layer F.SilkS)
+    (fp_text reference C6 (at 2.4892 0.127 90) (layer F.SilkS)
       (effects (font (size 1 1) (thickness 0.15)))
     )
@@
     (tags capacitor)
     (attr smd)
-    (fp_text reference C8 (at 0 -1.43 90) (layer F.SilkS)
+    (fp_text reference C8 (at 2.5653 0.1016 90) (layer F.SilkS)
       (effects (font (size 1 1) (thickness 0.15)))
     )
@@
     (tags capacitor)
     (attr smd)
-    (fp_text reference C9 (at 0 -1.65) (layer F.SilkS)
+    (fp_text reference C9 (at 2.6947 -0.2032) (layer F.SilkS)
       (effects (font (size 1 1) (thickness 0.15)))
     )
@@
   )
   (module Connector_PinSocket_2.54mm:PinSocket_2x15_P2.54mm_Vertical (layer F.Cu)
-    (at 91.44 72.39)
+    (at 109.22 72.39)
     (descr "Through hole straight socket strip, 2x15, 2.54mm pitch, double cols (from Kicad 4.0.7), script generated")
     (tags "Through hole socket strip THT 2x15 2.54mm double row")
-    (fp_text reference J3 (at -1.27 -2.77) (layer F.SilkS)
+    (fp_text reference J3 (at 2.921 -0.0762) (layer F.SilkS)
       (effects (font (size 1 1) (thickness 0.15)))
     )
@@
       (net 6 GND))
     (pad 5 thru_hole oval (at 0 5.08) (size 1.7 1.7) (drill 1) (layers *.Cu *.Mask)
-      (net 18 RST))
+      (net 40 RST1))
     (pad 6 thru_hole oval (at -2.54 5.08) (size 1.7 1.7) (drill 1) (layers *.Cu *.Mask)
-      (net 18 RST))
+      (net 40 RST1))
     (pad 7 thru_hole oval (at 0 7.62) (size 1.7 1.7) (drill 1) (layers *.Cu *.Mask)
       (net 7 5V))
@@
     (tags resistor)
     (attr smd)
-    (fp_text reference R1 (at 0 -1.43) (layer F.SilkS)
+    (fp_text reference R1 (at -2.4891 -0.0254) (layer F.SilkS)
       (effects (font (size 1 1) (thickness 0.15)))
     )
@@
     (tags resistor)
     (attr smd)
-    (fp_text reference R2 (at 0 -1.43) (layer F.SilkS)
+    (fp_text reference R2 (at -2.3876 0.1016) (layer F.SilkS)
       (effects (font (size 1 1) (thickness 0.15)))
     )
@@
     (descr "Generic Phoenix Contact connector footprint for: MCV_1,5/4-G-3.5; number of pins: 04; pin pitch: 3.50mm; Vertical || order number: 1843622 8A 160V")
     (tags "phoenix_contact connector MCV_01x04_G_3.5mm")
-    (fp_text reference J1 (at 5.25 -5.45 90) (layer F.SilkS)
+    (fp_text reference J1 (at 5.1712 4.3688 90) (layer F.SilkS)
       (effects (font (size 1 1) (thickness 0.15)))
     )
@@
     (descr "Generic Phoenix Contact connector footprint for: MCV_1,5/2-G-3.5; number of pins: 02; pin pitch: 3.50mm; Vertical || order number: 1843606 8A 160V")
     (tags "phoenix_contact connector MCV_01x02_G_3.5mm")
-    (fp_text reference J4 (at 1.75 -5.45 90) (layer F.SilkS)
+    (fp_text reference J4 (at 1.9558 4.2672 90) (layer F.SilkS)
       (effects (font (size 1 1) (thickness 0.15)))
     )
@@
     (descr "Generic Phoenix Contact connector footprint for: MCV_1,5/3-G-3.5; number of pins: 03; pin pitch: 3.50mm; Vertical || order number: 1843619 8A 160V")
     (tags "phoenix_contact connector MCV_01x03_G_3.5mm")
-    (fp_text reference J5 (at 3.5 -5.45 90) (layer F.SilkS)
+    (fp_text reference J5 (at 3.8608 4.3688 90) (layer F.SilkS)
       (effects (font (size 1 1) (thickness 0.15)))
     )
@@
     )
   )
-  (segment (start 88.9 74.93) (end 91.44 74.93) (width 0.25) (layer F.Cu) (net 6))
-  (segment (start 106.68 80.01) (end 109.22 80.01) (width 0.25) (layer F.Cu) (net 6))
-  (segment (start 88.9 80.01) (end 91.44 80.01) (width 0.25) (layer F.Cu) (net 7))
-  (segment (start 90.102081 72.39) (end 91.44 72.39) (width 0.25) (layer F.Cu) (net 8))
-  (segment (start 88.9 72.39) (end 90.102081 72.39) (width 0.25) (layer F.Cu) (net 8))
-  (segment (start 90.102081 105.41) (end 91.44 105.41) (width 0.25) (layer F.Cu) (net 9))
-  (segment (start 88.9 105.41) (end 90.102081 105.41) (width 0.25) (layer F.Cu) (net 9))
-  (segment (start 109.22 72.39) (end 106.68 72.39) (width 0.25) (layer F.Cu) (net 16))
-  (segment (start 106.68 74.93) (end 109.22 74.93) (width 0.25) (layer F.Cu) (net 17))
-  (segment (start 88.9 77.47) (end 91.44 77.47) (width 0.25) (layer F.Cu) (net 18))
-  (segment (start 109.22 77.47) (end 106.68 77.47) (width 0.25) (layer F.Cu) (net 18))
-  (segment (start 109.22 82.55) (end 106.68 82.55) (width 0.25) (layer F.Cu) (net 19))
-  (segment (start 106.68 85.09) (end 109.22 85.09) (width 0.25) (layer F.Cu) (net 20))
-  (segment (start 109.22 87.63) (end 106.68 87.63) (width 0.25) (layer F.Cu) (net 21))
-  (segment (start 106.68 90.17) (end 109.22 90.17) (width 0.25) (layer F.Cu) (net 22))
-  (segment (start 109.22 92.71) (end 106.68 92.71) (width 0.25) (layer F.Cu) (net 23))
-  (segment (start 106.68 95.25) (end 109.22 95.25) (width 0.25) (layer F.Cu) (net 24))
-  (segment (start 109.22 97.79) (end 106.68 97.79) (width 0.25) (layer F.Cu) (net 25))
-  (segment (start 106.68 100.33) (end 109.22 100.33) (width 0.25) (layer F.Cu) (net 26))
-  (segment (start 109.22 102.87) (end 106.68 102.87) (width 0.25) (layer F.Cu) (net 27))
-  (segment (start 106.68 105.41) (end 109.22 105.41) (width 0.25) (layer F.Cu) (net 28))
-  (segment (start 109.22 107.95) (end 106.68 107.95) (width 0.25) (layer F.Cu) (net 29))
-  (segment (start 88.9 82.55) (end 91.44 82.55) (width 0.25) (layer F.Cu) (net 30))
-  (segment (start 88.9 85.09) (end 91.44 85.09) (width 0.25) (layer F.Cu) (net 31))
-  (segment (start 88.9 87.63) (end 91.44 87.63) (width 0.25) (layer F.Cu) (net 32))
-  (segment (start 88.9 90.17) (end 91.44 90.17) (width 0.25) (layer F.Cu) (net 33))
-  (segment (start 91.44 92.71) (end 88.9 92.71) (width 0.25) (layer F.Cu) (net 34))
-  (segment (start 88.9 95.25) (end 91.44 95.25) (width 0.25) (layer F.Cu) (net 35))
-  (segment (start 90.237919 97.79) (end 88.9 97.79) (width 0.25) (layer F.Cu) (net 36))
-  (segment (start 91.44 97.79) (end 90.237919 97.79) (width 0.25) (layer F.Cu) (net 36))
-  (segment (start 88.9 100.33) (end 91.44 100.33) (width 0.25) (layer F.Cu) (net 37))
-  (segment (start 91.44 102.87) (end 88.9 102.87) (width 0.25) (layer F.Cu) (net 38))
-  (segment (start 91.44 107.95) (end 88.9 107.95) (width 0.25) (layer F.Cu) (net 39))
+  (gr_line (start 121.285 70.231) (end 121.285 110.363) (layer Edge.Cuts) (width 0.05))
+  (gr_line (start 86.7918 70.231) (end 121.285 70.231) (layer Edge.Cuts) (width 0.05))
+  (gr_line (start 86.741 110.363) (end 86.7918 70.231) (layer Edge.Cuts) (width 0.05))
+  (gr_line (start 121.285 110.363) (end 86.741 110.363) (layer Edge.Cuts) (width 0.05))
 )
