File: board/PCB_Bot.kicad_pcb (KiCad board)
At the start: 2 copper layers, 34.5 x 40.1 mm, 19 parts, among them J1 Screw_Terminal_01x04, J2 Conn_02x15_Top_Bottom, J3 Conn_02x15_Top_Bottom, J4 Screw_Terminal_01x02, J5 Conn_02x03_Top_Bottom, U1 TB6612FNG, U2 LSM9DS1

Commit message: add stp files and update boardlayoutex.md
Parts:
- removed A1: Arduino_Nano_v3.x, Module:Arduino_Nano
Changed lines of the file:
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@@
     (tracks 104)
     (zones 0)
-    (modules 19)
-    (nets 71)
+    (modules 18)
+    (nets 41)
   )
   (page A4)
@@
   (net 39 D13)
   (net 40 RST1)
-  (net 41 "Net-(A1-Pad1)")
-  (net 42 "Net-(A1-Pad17)")
-  (net 43 "Net-(A1-Pad2)")
-  (net 44 "Net-(A1-Pad18)")
-  (net 45 "Net-(A1-Pad3)")
-  (net 46 "Net-(A1-Pad19)")
-  (net 47 "Net-(A1-Pad4)")
-  (net 48 "Net-(A1-Pad20)")
-  (net 49 "Net-(A1-Pad5)")
-  (net 50 "Net-(A1-Pad21)")
-  (net 51 "Net-(A1-Pad6)")
-  (net 52 "Net-(A1-Pad22)")
-  (net 53 "Net-(A1-Pad7)")
-  (net 54 "Net-(A1-Pad23)")
-  (net 55 "Net-(A1-Pad8)")
-  (net 56 "Net-(A1-Pad24)")
-  (net 57 "Net-(A1-Pad9)")
-  (net 58 "Net-(A1-Pad25)")
-  (net 59 "Net-(A1-Pad10)")
-  (net 60 "Net-(A1-Pad26)")
-  (net 61 "Net-(A1-Pad11)")
-  (net 62 "Net-(A1-Pad27)")
-  (net 63 "Net-(A1-Pad12)")
-  (net 64 "Net-(A1-Pad28)")
-  (net 65 "Net-(A1-Pad13)")
-  (net 66 "Net-(A1-Pad29)")
-  (net 67 "Net-(A1-Pad14)")
-  (net 68 "Net-(A1-Pad30)")
-  (net 69 "Net-(A1-Pad15)")
-  (net 70 "Net-(A1-Pad16)")
   (net_class Default "This is the default net class."
     (clearance 0.2)
@@
     (add_net D9)
     (add_net GND)
-    (add_net "Net-(A1-Pad1)")
-    (add_net "Net-(A1-Pad10)")
-    (add_net "Net-(A1-Pad11)")
-    (add_net "Net-(A1-Pad12)")
-    (add_net "Net-(A1-Pad13)")
-    (add_net "Net-(A1-Pad14)")
-    (add_net "Net-(A1-Pad15)")
-    (add_net "Net-(A1-Pad16)")
-    (add_net "Net-(A1-Pad17)")
-    (add_net "Net-(A1-Pad18)")
-    (add_net "Net-(A1-Pad19)")
-    (add_net "Net-(A1-Pad2)")
-    (add_net "Net-(A1-Pad20)")
-    (add_net "Net-(A1-Pad21)")
-    (add_net "Net-(A1-Pad22)")
-    (add_net "Net-(A1-Pad23)")
-    (add_net "Net-(A1-Pad24)")
-    (add_net "Net-(A1-Pad25)")
-    (add_net "Net-(A1-Pad26)")
-    (add_net "Net-(A1-Pad27)")
-    (add_net "Net-(A1-Pad28)")
-    (add_net "Net-(A1-Pad29)")
-    (add_net "Net-(A1-Pad3)")
-    (add_net "Net-(A1-Pad30)")
-    (add_net "Net-(A1-Pad4)")
-    (add_net "Net-(A1-Pad5)")
-    (add_net "Net-(A1-Pad6)")
-    (add_net "Net-(A1-Pad7)")
-    (add_net "Net-(A1-Pad8)")
-    (add_net "Net-(A1-Pad9)")
     (add_net "Net-(C8-Pad1)")
     (add_net "Net-(C9-Pad1)")
@@
     (model ${KIPRJMOD}/Rnanobot.pretty/pxc_1815264_01_PTSM-0-5-2-HV-2-5-THR-WH-R32_3D_nocap.stp
       (offset (xyz -3.35 2.5 7.55))
+      (scale (xyz 1 1 1))
+      (rotate (xyz -90 -90 90))
+    )
+    (model ${KIPRJMOD}/Rnanobot.pretty/pxc_1704853_00_PTSM-0-5-2-P-2-5-WH_3D.stp
+      (offset (xyz -2.6 2.5 7.55))
       (scale (xyz 1 1 1))
       (rotate (xyz -90 -90 90))
@@
       (at (xyz 0 0 0))
       (scale (xyz 1 1 1))
-      (rotate (xyz 0 0 0))
-    )
-  )
-  (module Module:Arduino_Nano (layer F.Cu)
-    (at 62.29604 72.53732)
-    (descr "Arduino Nano, http://www.mouser.com/pdfdocs/Gravitech_Arduino_Nano3_0.pdf")
-    (tags "Arduino Nano")
-    (fp_text reference A1 (at 7.62 -5.08) (layer F.SilkS)
-      (effects (font (size 1 1) (thickness 0.15)))
-    )
-    (fp_text value Arduino_Nano_v3.x (at 8.89 19.05 90) (layer F.Fab)
-      (effects (font (size 1 1) (thickness 0.15)))
-    )
-    (fp_text user %R (at 6.35 19.05 90) (layer F.Fab)
-      (effects (font (size 1 1) (thickness 0.15)))
-    )
-    (fp_line (start 1.27 1.27) (end 1.27 -1.27) (layer F.SilkS) (width 0.12))
-    (fp_line (start 1.27 -1.27) (end -1.4 -1.27) (layer F.SilkS) (width 0.12))
-    (fp_line (start -1.4 1.27) (end -1.4 39.5) (layer F.SilkS) (width 0.12))
-    (fp_line (start -1.4 -3.94) (end -1.4 -1.27) (layer F.SilkS) (width 0.12))
-    (fp_line (start 13.97 -1.27) (end 16.64 -1.27) (layer F.SilkS) (width 0.12))
-    (fp_line (start 13.97 -1.27) (end 13.97 36.83) (layer F.SilkS) (width 0.12))
-    (fp_line (start 13.97 36.83) (end 16.64 36.83) (layer F.SilkS) (width 0.12))
-    (fp_line (start 1.27 1.27) (end -1.4 1.27) (layer F.SilkS) (width 0.12))
-    (fp_line (start 1.27 1.27) (end 1.27 36.83) (layer F.SilkS) (width 0.12))
-    (fp_line (start 1.27 36.83) (end -1.4 36.83) (layer F.SilkS) (width 0.12))
-    (fp_line (start 3.81 31.75) (end 11.43 31.75) (layer F.Fab) (width 0.1))
-    (fp_line (start 11.43 31.75) (end 11.43 41.91) (layer F.Fab) (width 0.1))
-    (fp_line (start 11.43 41.91) (end 3.81 41.91) (layer F.Fab) (width 0.1))
-    (fp_line (start 3.81 41.91) (end 3.81 31.75) (layer F.Fab) (width 0.1))
-    (fp_line (start -1.4 39.5) (end 16.64 39.5) (layer F.SilkS) (width 0.12))
-    (fp_line (start 16.64 39.5) (end 16.64 -3.94) (layer F.SilkS) (width 0.12))
-    (fp_line (start 16.64 -3.94) (end -1.4 -3.94) (layer F.SilkS) (width 0.12))
-    (fp_line (start 16.51 39.37) (end -1.27 39.37) (layer F.Fab) (width 0.1))
-    (fp_line (start -1.27 39.37) (end -1.27 -2.54) (layer F.Fab) (width 0.1))
-    (fp_line (start -1.27 -2.54) (end 0 -3.81) (layer F.Fab) (width 0.1))
-    (fp_line (start 0 -3.81) (end 16.51 -3.81) (layer F.Fab) (width 0.1))
-    (fp_line (start 16.51 -3.81) (end 16.51 39.37) (layer F.Fab) (width 0.1))
-    (fp_line (start -1.53 -4.06) (end 16.75 -4.06) (layer F.CrtYd) (width 0.05))
-    (fp_line (start -1.53 -4.06) (end -1.53 42.16) (layer F.CrtYd) (width 0.05))
-    (fp_line (start 16.75 42.16) (end 16.75 -4.06) (layer F.CrtYd) (width 0.05))
-    (fp_line (start 16.75 42.16) (end -1.53 42.16) (layer F.CrtYd) (width 0.05))
-    (pad 1 thru_hole rect (at 0 0) (size 1.6 1.6) (drill 0.8) (layers *.Cu *.Mask)
-      (net 41 "Net-(A1-Pad1)"))
-    (pad 17 thru_hole oval (at 15.24 33.02) (size 1.6 1.6) (drill 0.8) (layers *.Cu *.Mask)
-      (net 42 "Net-(A1-Pad17)"))
-    (pad 2 thru_hole oval (at 0 2.54) (size 1.6 1.6) (drill 0.8) (layers *.Cu *.Mask)
-      (net 43 "Net-(A1-Pad2)"))
-    (pad 18 thru_hole oval (at 15.24 30.48) (size 1.6 1.6) (drill 0.8) (layers *.Cu *.Mask)
-      (net 44 "Net-(A1-Pad18)"))
-    (pad 3 thru_hole oval (at 0 5.08) (size 1.6 1.6) (drill 0.8) (layers *.Cu *.Mask)
-      (net 45 "Net-(A1-Pad3)"))
-    (pad 19 thru_hole oval (at 15.24 27.94) (size 1.6 1.6) (drill 0.8) (layers *.Cu *.Mask)
-      (net 46 "Net-(A1-Pad19)"))
-    (pad 4 thru_hole oval (at 0 7.62) (size 1.6 1.6) (drill 0.8) (layers *.Cu *.Mask)
-      (net 47 "Net-(A1-Pad4)"))
-    (pad 20 thru_hole oval (at 15.24 25.4) (size 1.6 1.6) (drill 0.8) (layers *.Cu *.Mask)
-      (net 48 "Net-(A1-Pad20)"))
-    (pad 5 thru_hole oval (at 0 10.16) (size 1.6 1.6) (drill 0.8) (layers *.Cu *.Mask)
-      (net 49 "Net-(A1-Pad5)"))
-    (pad 21 thru_hole oval (at 15.24 22.86) (size 1.6 1.6) (drill 0.8) (layers *.Cu *.Mask)
-      (net 50 "Net-(A1-Pad21)"))
-    (pad 6 thru_hole oval (at 0 12.7) (size 1.6 1.6) (drill 0.8) (layers *.Cu *.Mask)
-      (net 51 "Net-(A1-Pad6)"))
-    (pad 22 thru_hole oval (at 15.24 20.32) (size 1.6 1.6) (drill 0.8) (layers *.Cu *.Mask)
-      (net 52 "Net-(A1-Pad22)"))
-    (pad 7 thru_hole oval (at 0 15.24) (size 1.6 1.6) (drill 0.8) (layers *.Cu *.Mask)
-      (net 53 "Net-(A1-Pad7)"))
-    (pad 23 thru_hole oval (at 15.24 17.78) (size 1.6 1.6) (drill 0.8) (layers *.Cu *.Mask)
-      (net 54 "Net-(A1-Pad23)"))
-    (pad 8 thru_hole oval (at 0 17.78) (size 1.6 1.6) (drill 0.8) (layers *.Cu *.Mask)
-      (net 55 "Net-(A1-Pad8)"))
-    (pad 24 thru_hole oval (at 15.24 15.24) (size 1.6 1.6) (drill 0.8) (layers *.Cu *.Mask)
-      (net 56 "Net-(A1-Pad24)"))
-    (pad 9 thru_hole oval (at 0 20.32) (size 1.6 1.6) (drill 0.8) (layers *.Cu *.Mask)
-      (net 57 "Net-(A1-Pad9)"))
-    (pad 25 thru_hole oval (at 15.24 12.7) (size 1.6 1.6) (drill 0.8) (layers *.Cu *.Mask)
-      (net 58 "Net-(A1-Pad25)"))
-    (pad 10 thru_hole oval (at 0 22.86) (size 1.6 1.6) (drill 0.8) (layers *.Cu *.Mask)
-      (net 59 "Net-(A1-Pad10)"))
-    (pad 26 thru_hole oval (at 15.24 10.16) (size 1.6 1.6) (drill 0.8) (layers *.Cu *.Mask)
-      (net 60 "Net-(A1-Pad26)"))
-    (pad 11 thru_hole oval (at 0 25.4) (size 1.6 1.6) (drill 0.8) (layers *.Cu *.Mask)
-      (net 61 "Net-(A1-Pad11)"))
-    (pad 27 thru_hole oval (at 15.24 7.62) (size 1.6 1.6) (drill 0.8) (layers *.Cu *.Mask)
-      (net 62 "Net-(A1-Pad27)"))
-    (pad 12 thru_hole oval (at 0 27.94) (size 1.6 1.6) (drill 0.8) (layers *.Cu *.Mask)
-      (net 63 "Net-(A1-Pad12)"))
-    (pad 28 thru_hole oval (at 15.24 5.08) (size 1.6 1.6) (drill 0.8) (layers *.Cu *.Mask)
-      (net 64 "Net-(A1-Pad28)"))
-    (pad 13 thru_hole oval (at 0 30.48) (size 1.6 1.6) (drill 0.8) (layers *.Cu *.Mask)
-      (net 65 "Net-(A1-Pad13)"))
-    (pad 29 thru_hole oval (at 15.24 2.54) (size 1.6 1.6) (drill 0.8) (layers *.Cu *.Mask)
-      (net 66 "Net-(A1-Pad29)"))
-    (pad 14 thru_hole oval (at 0 33.02) (size 1.6 1.6) (drill 0.8) (layers *.Cu *.Mask)
-      (net 67 "Net-(A1-Pad14)"))
-    (pad 30 thru_hole oval (at 15.24 0) (size 1.6 1.6) (drill 0.8) (layers *.Cu *.Mask)
-      (net 68 "Net-(A1-Pad30)"))
-    (pad 15 thru_hole oval (at 0 35.56) (size 1.6 1.6) (drill 0.8) (layers *.Cu *.Mask)
-      (net 69 "Net-(A1-Pad15)"))
-    (pad 16 thru_hole oval (at 15.24 35.56) (size 1.6 1.6) (drill 0.8) (layers *.Cu *.Mask)
-      (net 70 "Net-(A1-Pad16)"))
-    (model ${KISYS3DMOD}/Module.3dshapes/Arduino_Nano_WithMountingHoles.wrl
-      (at (xyz 0 0 0))
-      (scale (xyz 1 1 1))
